Commit message: Add possibility to adjust HAP sample number

File: urdf/HAP.xacro (robot description, xacro)
@@ -4,5 +4,5 @@
   <xacro:property name="laser_min_range" value="0.1"/>
   <xacro:property name="laser_max_range" value="200.0"/>
-  <xacro:property name="samples" value="45300"/>
+  <xacro:property name="samples" value="$(optenv GZB_LIVOX_SAMPLES)"/>
   <xacro:property name="resolution" value="0.002"/>
   <xacro:property name="noise_mean" value="0.0"/>
@@ -66,4 +66,8 @@
 			  </noise>
 			</ray>
+			<ros>
+                          <remapping>${topic}:=None</remapping>
+                          <remapping>${topic}_PointCloud2:=${topic}</remapping>
+             		</ros>
           <visualize>false</visualize>
 		  <samples>${samples}</samples>
